File: projects/MorsePrototype/MorsePrototype.kicad_pcb (KiCad board)
At the start: 2 copper layers, 65 x 51 mm, 50 parts, among them J1 Audio Out Jack, J2 Paddle Jack, P1 UART, P2 SBW JTAG, P3 Power, U1 OPA4322, U2 OPA322, U3 TS5A2066, U4 MSP430G2x53, U5 SN74AHC1G32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

Commit message: 170329 Update
Parts:
- R10, R12, R13, R14, R5, R6, R7, R8, R9: value 105k -> 47k
- R11: value 105k -> 470
- moved W1 6.08 mm to (170.5, 65.0)
- moved W4 1.50 mm to (163.0, 72.0)
- moved C1 1.00 mm to (168.0, 66.5)
- moved R1 1.00 mm to (165.5, 66.5)
- moved R5 1.00 mm to (165.5, 58.5)
- moved R6 1.00 mm to (168.0, 58.5)
- moved RF1 1.00 mm to (165.5, 73.5)
- moved RG1 1.00 mm to (168.0, 73.5)
- turned U2 to 90 degrees
Connections:
- U1 pad 10: Net-(R3-Pad1) -> Net-(C2-Pad1)
- U1 pad 12: Net-(R4-Pad1) -> Net-(C3-Pad2)
- U1 pad 13: Net-(C3-Pad2) -> Net-(R4-Pad1)
- U1 pad 2: Net-(R5-Pad2) -> Net-(RF1-Pad1)
- U1 pad 3: Net-(RF1-Pad1) -> Net-(R5-Pad2)
- U1 pad 5: Net-(R2-Pad2) -> Net-(C1-Pad1)
- U1 pad 6: Net-(C1-Pad1) -> Net-(R2-Pad2)
- U1 pad 9: Net-(C2-Pad1) -> Net-(R3-Pad1)
- U2 pad 3: Net-(U2-Pad1) -> Net-(C4-Pad2)
- U2 pad 4: Net-(C4-Pad2) -> Net-(U2-Pad1)
Routing:
- net Net-(R4-Pad1): track 7.08 -> 3.30 mm
- net Net-(R2-Pad2): track 7.08 -> 3.30 mm
- net Net-(R5-Pad2): track 18.2 -> 22.0 mm
- net Net-(RF1-Pad1): track 12.5 -> 9.60 mm, vias 0 -> 2
- net Net-(R3-Pad1): track 6.48 -> 3.87 mm
- net Net-(R1-Pad2): track 16.6 -> 14.3 mm
- net Net-(C4-Pad2): track 15.1 -> 13.2 mm
- net GND: track 89.0 -> 90.6 mm
- net Net-(C2-Pad1): track 10.6 -> 11.2 mm
- net Net-(C1-Pad1): track 8.10 -> 8.63 mm
Other:
- outline, holes or cut-outs redrawn
- board text added: "Morse Oscillator Prototype 29 Mar 2017"
- board text removed: "Morse Oscillator Prototype 9 Mar 2017"
