File: projects/MorsePrototype/MorsePrototype.sch (KiCad schematic (older format))
At the start: 50 parts, among them J1 Audio Out Jack, J2 Paddle Jack, P1 UART, P2 SBW JTAG, P3 Power, U1 OPA4322, U2 OPA322, U3 TS5A2066, U4 MSP430G2x53, U5 SN74AHC1G32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

Commit message: 170329 Update
Parts:
- R10, R12, R13, R14, R5, R6, R7, R8, R9: value 105k -> 47k
- R11: value 105k -> 470
Connections:
- net at R5.2, R6.2: now also U1.3 (+); no longer U1.2 (-)
- net at RF1.1, RG1.1: now also U1.2 (-); no longer U1.3 (+)
- net at R2.2, U1.7: now also U1.6 (-); no longer U1.5 (+)
- net at C1.1, R1.1, W1.1: now also U1.5 (+); no longer U1.6 (-)
- net at R3.1, U1.8: now also U1.9 (-); no longer U1.10 (+)
- net at C2.1, R2.1, W2.1: now also U1.10 (+); no longer U1.9 (-)
- net at R4.1, U1.14: now also U1.13 (-); no longer U1.12 (+)
- net at C3.2, R3.2, W3.1: now also U1.12 (+); no longer U1.13 (-)
- net at C4.2, R4.2, RF1.2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: now also U2.3 (+); no longer U2.4 (-)
- net at U2.1, U3.1 (NO1), W5.1: now also U2.4 (-); no longer U2.3 (+)
Changed lines of the file:
@@
 F 3 "" H 2150 2750 50  0000 C CNN
 	1    2150 2750
-	1    0    0    -1
+	1    0    0    1
 $EndComp
 $Comp
@@
 F 3 "" H 3350 2750 50  0000 C CNN
 	2    3350 2750
-	1    0    0    -1
+	1    0    0    1
 $EndComp
 $Comp
@@
 F 3 "" H 4550 2750 50  0000 C CNN
 	3    4550 2750
-	1    0    0    -1
+	1    0    0    1
 $EndComp
 $Comp
@@
 F 3 "" H 5750 2750 50  0000 C CNN
 	4    5750 2750
-	1    0    0    -1
+	1    0    0    1
 $EndComp
 $Comp
@@
 P 1250 2650
 F 0 "R5" V 1330 2650 50  0000 C CNN
-F 1 "105k" V 1250 2650 50  0000 C CNN
+F 1 "47k" V 1250 2650 50  0000 C CNN
 F 2 "Resistors_SMD:R_0805_HandSoldering" V 1180 2650 50  0001 C CNN
 F 3 "" H 1250 2650 50  0000 C CNN
@@
 P 1250 3050
 F 0 "R6" V 1330 3050 50  0000 C CNN
-F 1 "105k" V 1250 3050 50  0000 C CNN
+F 1 "47k" V 1250 3050 50  0000 C CNN
 F 2 "Resistors_SMD:R_0805_HandSoldering" V 1180 3050 50  0001 C CNN
 F 3 "" H 1250 3050 50  0000 C CNN
@@
 F 3 "" H 6950 3000 50  0000 C CNN
 	1    6950 2750
-	1    0    0    -1
+	1    0    0    1
 $EndComp
 $Comp
@@
 P 4550 4800
 F 0 "R7" V 4630 4800 50  0000 C CNN
-F 1 "105k" V 4550 4800 50  0000 C CNN
+F 1 "47k" V 4550 4800 50  0000 C CNN
 F 2 "Resistors_SMD:R_0805_HandSoldering" V 4480 4800 50  0001 C CNN
 F 3 "" H 4550 4800 50  0000 C CNN
@@
 P 2500 6100
 F 0 "R12" V 2580 6100 50  0000 C CNN
-F 1 "105k" V 2500 6100 50  0000 C CNN
+F 1 "47k" V 2500 6100 50  0000 C CNN
 F 2 "Resistors_SMD:R_0805_HandSoldering" V 2430 6100 50  0001 C CNN
 F 3 "" H 2500 6100 50  0000 C CNN
@@
 P 5900 4850
 F 0 "R8" V 5980 4850 50  0000 C CNN
-F 1 "105k" V 5900 4850 50  0000 C CNN
+F 1 "47k" V 5900 4850 50  0000 C CNN
 F 2 "Resistors_SMD:R_0805_HandSoldering" V 5830 4850 50  0001 C CNN
 F 3 "" H 5900 4850 50  0000 C CNN
@@
 P 6250 4850
 F 0 "R9" V 6330 4850 50  0000 C CNN
-F 1 "105k" V 6250 4850 50  0000 C CNN
+F 1 "47k" V 6250 4850 50  0000 C CNN
 F 2 "Resistors_SMD:R_0805_HandSoldering" V 6180 4850 50  0001 C CNN
 F 3 "" H 6250 4850 50  0000 C CNN
@@
 P 6600 4850
 F 0 "R10" V 6680 4850 50  0000 C CNN
-F 1 "105k" V 6600 4850 50  0000 C CNN
+F 1 "47k" V 6600 4850 50  0000 C CNN
 F 2 "Resistors_SMD:R_0805_HandSoldering" V 6530 4850 50  0001 C CNN
 F 3 "" H 6600 4850 50  0000 C CNN
@@
 P 6950 4850
 F 0 "R11" V 7030 4850 50  0000 C CNN
-F 1 "105k" V 6950 4850 50  0000 C CNN
+F 1 "470" V 6950 4850 50  0000 C CNN
 F 2 "Resistors_SMD:R_0805_HandSoldering" V 6880 4850 50  0001 C CNN
 F 3 "" H 6950 4850 50  0000 C CNN
@@
 P 8650 4250
 F 0 "R13" V 8730 4250 50  0000 C CNN
-F 1 "105k" V 8650 4250 50  0000 C CNN
+F 1 "47k" V 8650 4250 50  0000 C CNN
 F 2 "Resistors_SMD:R_0805_HandSoldering" V 8580 4250 50  0001 C CNN
 F 3 "" H 8650 4250 50  0000 C CNN
@@
 P 8950 4250
 F 0 "R14" V 9030 4250 50  0000 C CNN
-F 1 "105k" V 8950 4250 50  0000 C CNN
+F 1 "47k" V 8950 4250 50  0000 C CNN
 F 2 "Resistors_SMD:R_0805_HandSoldering" V 8880 4250 50  0001 C CNN
 F 3 "" H 8950 4250 50  0000 C CNN
