File: projects/Si5351-2m_test/Si5351-2m.kicad_pcb (KiCad board)
At the start: 2 copper layers, 32 x 35 mm, 16 parts, among them P1 CONN_01X04, U1 Si5351A, X1 25 MHz

Commit message: 170907b Update
Parts:
- moved C2 6.52 mm to (144.5, 106.0), turned to 180 degrees
- moved L2 3.81 mm to (144.5, 104.0), turned to 0 degrees
- moved C3 2.92 mm to (146.5, 100.0)
- moved L3 2.55 mm to (143.5, 101.0), turned to 90 degrees
- moved C1 1.58 mm to (140.5, 104.0), turned to 180 degrees
- moved L1 0.71 mm to (139.5, 107.0), turned to 90 degrees
Routing:
- net Out1: track 9.47 -> 5.78 mm
- net Out2: track 17.3 -> 19.3 mm
- net Net-(C3-Pad2): track 2.79 -> 2.07 mm
- added copper zone on F.Cu, net Out2
Other:
- net class 50ohm: trace_width 2.97 -> 0.75
- board text added: "170428"
- board text removed: "170427"
