File: projects/Battery-Experiments/Avionics Battery Prototype/Avionics Battery Prototype.kicad_pcb (KiCad board)
At the start: 2 copper layers, 134 x 139.7 mm, 59 parts, among them J1 Jack-DC, J2 Enable, J3 UART, J4 SBW JTAG, U1 OPA4197, U2 OPA4197, U3 CD4052B, U4 LT1763, U5 MSP430G2233, U6 CD40109B

Commit message: Syncing AVB Rev C
Parts:
- added TP3: XTAL, k7arx:8MM-11 2-pin PCB socket, F.Cu at (147.3, 57.1)
Connections:
- U5 pad 18: GND -> /X-
- U5 pad 19: GND -> /X+
Routing:
- net /X-: track 0.00 -> 13.7 mm, vias 0 -> 1
- net /X+: track 0.00 -> 13.2 mm, vias 0 -> 1
- net GND: track 70.7 -> 59.9 mm, vias 2 -> 3
Other:
- board text added: "LFXTL"
