File: projects/Battery-Experiments/Avionics Battery Prototype/Avionics Battery Prototype.kicad_pcb (KiCad board)
At the start: 2 copper layers, 134 x 139.7 mm, 59 parts, among them J1 Jack-DC, J2 Enable, J3 UART, J4 SBW JTAG, U1 OPA4197, U2 OPA4197, U3 CD4052B, U4 LT1763, U5 MSP430G2233, U6 CD40109B

Commit message: Syncing AVB Rev C from Taran
Parts:
- J1: footprint Connect:Banana_Jack_2Pin -> k7arx:Anderson PowerPole PCB 2H1V
- moved J1 19.0 mm to (71.1, 167.6), turned to 180 degrees
Routing:
- net GND: track 70.7 -> 91.7 mm
- net Net-(J1-Pad1): track 67.0 -> 78.2 mm
Other:
- board text added: "Avionics Battery Prototype Rev C"
- board text removed: "Avionics Battery Prototype Rev B"
Changed lines of the file:
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@@
     (thickness 1.6)
     (drawings 21)
-    (tracks 427)
+    (tracks 429)
     (zones 0)
     (modules 59)
@@
   )
   (setup
-    (last_trace_width 0.3)
+    (last_trace_width 1.016)
     (user_trace_width 0.508)
     (user_trace_width 1.016)
@@
     (add_net ~RST)
   )
+  (module "k7arx:Anderson PowerPole PCB 2H1V" (layer F.Cu)
+    (at 71.12 167.64 180)
+    (fp_text reference J1 (at 9.525 13.97) (layer F.SilkS)
+      (effects (font (size 1 1) (thickness 0.15)))
+    )
+    (fp_text value Jack-DC (at 14.985 6.29) (layer F.Fab)
+      (effects (font (size 1 1) (thickness 0.15)))
+    )
+    (fp_text user %R (at 14.985 0) (layer F.Fab)
+      (effects (font (size 1 1) (thickness 0.15)))
+    )
+    (fp_line (start 7.39 14.7) (end 7.39 0) (layer F.SilkS) (width 0.25))
+    (fp_line (start -7.39 14.7) (end 7.39 14.7) (layer F.SilkS) (width 0.25))
+    (fp_line (start -7.39 0) (end -7.39 14.7) (layer F.SilkS) (width 0.25))
+    (fp_line (start 7.39 0) (end -7.39 0) (layer F.SilkS) (width 0.25))
+    (pad "" np_thru_hole circle (at -12.155 7.32 180) (size 5.57 5.57) (drill 4.57) (layers *.Cu *.Mask))
+    (pad "" np_thru_hole circle (at 12.155 7.32 180) (size 5.57 5.57) (drill 4.57) (layers *.Cu *.Mask))
+    (pad 1 thru_hole oval (at -3.95 18.24 180) (size 6.23 2.27) (drill oval 5.23 1.27) (layers *.Cu *.Mask)
+      (net 47 "Net-(J1-Pad1)"))
+    (pad 2 thru_hole oval (at 3.95 18.24 180) (size 6.23 2.27) (drill oval 5.23 1.27) (layers *.Cu *.Mask)
+      (net 2 GND))
+  )
   (module k7arx:K7ARX-10mm (layer F.Cu)
     (at 137.16 119.38)
@@
       (xy 16.181075 -4.785006)) (layer F.Mask) (width 0.01))
   )
-  (module Connect:Banana_Jack_2Pin (layer F.Cu)
-    (at 55.88 156.21)
-    (descr "Dual banana socket, footprint - 2 x 6mm drills")
-    (tags "banana socket")
-    (fp_text reference J1 (at 14.985 -6.604) (layer F.SilkS)
-      (effects (font (size 1 1) (thickness 0.15)))
-    )
-    (fp_text value Jack-DC (at 14.985 6.29) (layer F.Fab)
-      (effects (font (size 1 1) (thickness 0.15)))
-    )
-    (fp_line (start 30 -5.5) (end 0 -5.5) (layer F.CrtYd) (width 0.05))
-    (fp_line (start 0 5.5) (end 30 5.5) (layer F.CrtYd) (width 0.05))
-    (fp_line (start 0 5.25) (end 30 5.25) (layer F.SilkS) (width 0.12))
-    (fp_line (start 30 -5.25) (end 0 -5.25) (layer F.SilkS) (width 0.12))
-    (fp_circle (center 30 0) (end 32 0) (layer F.Fab) (width 0.1))
-    (fp_circle (center 0 0) (end 2 0) (layer F.Fab) (width 0.1))
-    (fp_circle (center 0 0) (end 4.75 0) (layer F.Fab) (width 0.1))
-    (fp_circle (center 30 0) (end 34.75 0) (layer F.Fab) (width 0.1))
-    (fp_arc (start 0 0) (end 0 5.25) (angle 180) (layer F.SilkS) (width 0.12))
-    (fp_arc (start 30 0) (end 30 -5.25) (angle 180) (layer F.SilkS) (width 0.12))
-    (fp_arc (start 30 0) (end 30 -5.5) (angle 180) (layer F.CrtYd) (width 0.05))
-    (fp_arc (start 0 0) (end 0 5.5) (angle 180) (layer F.CrtYd) (width 0.05))
-    (fp_text user %R (at 14.985 0) (layer F.Fab)
-      (effects (font (size 1 1) (thickness 0.15)))
-    )
-    (pad 2 thru_hole circle (at 29.97 0) (size 10.16 10.16) (drill 6.1) (layers *.Cu *.Mask)
-      (net 2 GND))
-    (pad 1 thru_hole circle (at 0 0) (size 10.16 10.16) (drill 6.1) (layers *.Cu *.Mask)
-      (net 47 "Net-(J1-Pad1)"))
-    (model ${KISYS3DMOD}/Connectors.3dshapes/Banana_Jack_2Pin.wrl
-      (offset (xyz 14.98599977493286 0 0))
-      (scale (xyz 2 2 2))
-      (rotate (xyz 0 0 0))
-    )
-  )
   (module Pin_Headers:Pin_Header_Straight_1x02_Pitch2.54mm (layer F.Cu)
     (at 99.06 137.16 180)
@@
   (gr_arc (start 168.91 163.83) (end 168.91 167.64) (angle -90) (layer Edge.Cuts) (width 0.05))
   (gr_arc (start 168.91 31.75) (end 172.72 31.75) (angle -90) (layer Edge.Cuts) (width 0.05))
-  (gr_text "Avionics Battery Prototype Rev B" (at 137.16 129.54) (layer F.Cu)
+  (gr_text "Avionics Battery Prototype Rev C" (at 137.16 129.54) (layer F.Cu)
     (effects (font (size 1.905 1.524) (thickness 0.254)))
   )
@@
   (segment (start 136.6774 54.483) (end 136.6774 53.1114) (width 0.3) (layer F.Cu) (net 2))
   (segment (start 135.255 33.655) (end 133.985 33.655) (width 0.3) (layer F.Cu) (net 2))
-  (segment (start 85.85 156.21) (end 105.41 156.21) (width 2.032) (layer F.Cu) (net 2))
+  (segment (start 67.17 149.4) (end 67.17 152.26) (width 2.032) (layer F.Cu) (net 2))
+  (segment (start 67.17 152.26) (end 70.485 155.575) (width 2.032) (layer F.Cu) (net 2))
+  (segment (start 70.485 155.575) (end 103.505 155.575) (width 2.032) (layer F.Cu) (net 2))
   (segment (start 105.918 82.55) (end 103.285 82.55) (width 0.508) (layer F.Cu) (net 3))
   (segment (start 103.285 82.55) (end 91.855 93.98) (width 0.508) (layer F.Cu) (net 3))
@@
   (segment (start 140.660202 58.42) (end 126.7635 58.42) (width 0.3) (layer F.Cu) (net 45))
   (segment (start 125.73 59.4535) (end 125.73 60.325) (width 0.3) (layer F.Cu) (net 45))
+  (segment (start 75.07 143.65) (end 75.07 149.4) (width 2.032) (layer F.Cu) (net 47))
+  (segment (start 71.53 140.11) (end 75.07 143.65) (width 2.032) (layer F.Cu) (net 47))
+  (segment (start 54.435 140.11) (end 71.53 140.11) (width 2.032) (layer F.Cu) (net 47))
   (segment (start 99.06 137.16) (end 54.61 137.16) (width 1.016) (layer F.Cu) (net 47))
   (segment (start 54.435 134.21) (end 54.435 140.11) (width 2.032) (layer F.Cu) (net 47))
-  (segment (start 54.435 140.11) (end 54.435 144.605) (width 2.032) (layer F.Cu) (net 47))
-  (segment (start 55.88 146.05) (end 55.88 156.21) (width 2.032) (layer F.Cu) (net 47))
-  (segment (start 54.435 144.605) (end 55.88 146.05) (width 2.032) (layer F.Cu) (net 47))
   (zone (net 2) (net_name GND) (layer F.Cu) (hatch edge 0.508)
     (connect_pads (clearance 0.508))
