File: projects/Battery-Experiments/Avionics Battery Prototype/Avionics Battery Prototype.sch (KiCad schematic (older format))
At the start: 60 parts, among them J1 Jack-DC, J2 Enable, J3 UART, J4 SBW JTAG, U1 OPA4197, U2 OPA4197, U3 CD4052B, U4 LT1763, U5 MSP430G2233, U6 CD40109B

Commit message: Syncing AVB Rev C
Parts:
- removed TP3: Xin, Pin_Headers:Pin_Header_Straight_1x01_Pitch2.54mm, symbol Connector:Conn_01x01_Female
- removed TP4: Xout, Pin_Headers:Pin_Header_Straight_1x01_Pitch2.54mm, symbol Connector:Conn_01x01_Female
- added TP3: XTAL, k7arx:8MM-11 2-pin PCB socket, symbol Connector_Generic:Conn_01x02
Connections:
- net X+: now reaches U5.19 (XIn)
- net X+: now also TP3.1 (Pin_1)
- net X-: now reaches U5.18 (XOut)
- net X-: now also TP3.2 (Pin_2)
Changed lines of the file:
@@
 Wire Wire Line
 	2800 2600 2900 2600
+Wire Wire Line
+	2800 3000 3600 3000
 $Comp
-L Connector:Conn_01x01_Female TP3
-U 1 1 6061AE7F
-P 3300 2700
-F 0 "TP3" H 3328 2726 50  0000 L CNN
-F 1 "Xin" H 3350 2800 50  0000 L CNN
-F 2 "Pin_Headers:Pin_Header_Straight_1x01_Pitch2.54mm" H 3300 2700 50  0001 C CNN
-F 3 "~" H 3300 2700 50  0001 C CNN
-	1    3300 2700
-	1    0    0    -1
-$EndComp
-$Comp
-L Connector:Conn_01x01_Female TP4
-U 1 1 6061B8E9
-P 3300 2800
-F 0 "TP4" H 3328 2826 50  0000 L CNN
-F 1 "Xout" H 3328 2735 50  0000 L CNN
-F 2 "Pin_Headers:Pin_Header_Straight_1x01_Pitch2.54mm" H 3300 2800 50  0001 C CNN
-F 3 "~" H 3300 2800 50  0001 C CNN
-	1    3300 2800
+L Connector_Generic:Conn_01x02 TP3
+U 1 1 604B2441
+P 3250 2700
+F 0 "TP3" H 3330 2692 50  0000 L CNN
+F 1 "XTAL" H 3330 2601 50  0000 L CNN
+F 2 "k7arx:8MM-11 2-pin PCB socket" H 3250 2700 50  0001 C CNN
+F 3 "~" H 3250 2700 50  0001 C CNN
+	1    3250 2700
 	1    0    0    -1
 $EndComp
 Wire Wire Line
-	2800 3000 3600 3000
+	2800 2700 3050 2700
 Wire Wire Line
-	2800 2700 3100 2700
-Wire Wire Line
-	2800 2800 3100 2800
+	2800 2800 3050 2800
+Text Label 2850 2700 0    50   ~ 0
+X+
+Text Label 2850 2800 0    50   ~ 0
+X-
 $EndSCHEMATC
