File: projects/Battery-Experiments/Avionics Battery Prototype/Avionics Battery Prototype.sch (KiCad schematic (older format))
At the start: 59 parts, among them J1 Jack-DC, J2 Enable, J3 UART, J4 SBW JTAG, U1 OPA4197, U2 OPA4197, U3 CD4052B, U4 LT1763, U5 MSP430G2233, U6 CD40109B

Commit message: AVB Rev C Final
Parts:
- J1: footprint Connect:Banana_Jack_2Pin -> k7arx:Anderson_PowerPole_PCB_2H1V
Changed lines of the file:
@@
 F 0 "J1" H 5757 1525 50  0000 C CNN
 F 1 "Jack-DC" H 5757 1434 50  0000 C CNN
-F 2 "Connect:Banana_Jack_2Pin" H 5750 1160 50  0001 C CNN
+F 2 "k7arx:Anderson_PowerPole_PCB_2H1V" H 5750 1160 50  0001 C CNN
 F 3 "~" H 5750 1160 50  0001 C CNN
 	1    5700 1200
