File: projects/Battery-Experiments/Avionics Battery Prototype/Avionics Battery Prototype - Rev C.kicad_pcb (KiCad board)
At the start: 2 copper layers, 134 x 139.7 mm, 60 parts, among them J1 Jack-DC, J2 Enable, J3 UART, J4 SBW JTAG, U1 OPA4197, U2 OPA4197, U3 CD4052B, U4 LT1763, U5 MSP430G2233, U6 CD40109B

Commit message: AVB Rev C Final
Routing:
- net GND: track 77.3 -> 67.2 mm
- net Net-(J1-Pad1): track 79.5 -> 71.0 mm
Changed lines of the file:
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@@
     (thickness 1.6)
     (drawings 22)
-    (tracks 434)
+    (tracks 430)
     (zones 0)
     (modules 60)
@@
     (add_net ~RST)
   )
+  (module k7arx:Anderson_PowerPole_PCB_2H1V (layer F.Cu)
+    (at 71.12 167.64 180)
+    (fp_text reference J1 (at 8.89 13.97) (layer F.SilkS)
+      (effects (font (size 1 1) (thickness 0.15)))
+    )
+    (fp_text value Jack-DC (at 0 16) (layer F.Fab)
+      (effects (font (size 1 1) (thickness 0.15)))
+    )
+    (fp_line (start 7.39 14.7) (end 7.39 0) (layer F.SilkS) (width 0.25))
+    (fp_line (start -7.39 14.7) (end 7.39 14.7) (layer F.SilkS) (width 0.25))
+    (fp_line (start -7.39 0) (end -7.39 14.7) (layer F.SilkS) (width 0.25))
+    (fp_line (start 7.39 0) (end -7.39 0) (layer F.SilkS) (width 0.25))
+    (pad 1 thru_hole circle (at 3.95 15.8 180) (size 3 3) (drill 1.8) (layers *.Cu *.Mask)
+      (net 47 "Net-(J1-Pad1)"))
+    (pad 2 thru_hole circle (at -3.95 15.8 180) (size 3 3) (drill 1.8) (layers *.Cu *.Mask)
+      (net 2 GND))
+    (pad "" np_thru_hole circle (at 12.155 7.32 180) (size 5.57 5.57) (drill 4.57) (layers *.Cu *.Mask))
+    (pad "" np_thru_hole circle (at -12.155 7.32 180) (size 5.57 5.57) (drill 4.57) (layers *.Cu *.Mask))
+  )
   (module "k7arx:8MM-11 2-pin PCB socket" (layer F.Cu)
     (at 147.32 57.15 270)
@@
     )
   )
-  (module k7arx:Anderson_PowerPole_PCB_2H1V (layer F.Cu)
-    (at 71.12 167.64 180)
-    (fp_text reference J1 (at 8.89 13.97) (layer F.SilkS)
-      (effects (font (size 1 1) (thickness 0.15)))
-    )
-    (fp_text value Jack-DC (at 0 16) (layer F.Fab)
-      (effects (font (size 1 1) (thickness 0.15)))
-    )
-    (fp_line (start 7.39 14.7) (end 7.39 0) (layer F.SilkS) (width 0.25))
-    (fp_line (start -7.39 14.7) (end 7.39 14.7) (layer F.SilkS) (width 0.25))
-    (fp_line (start -7.39 0) (end -7.39 14.7) (layer F.SilkS) (width 0.25))
-    (fp_line (start 7.39 0) (end -7.39 0) (layer F.SilkS) (width 0.25))
-    (pad "" np_thru_hole circle (at -12.155 7.32 180) (size 5.57 5.57) (drill 4.57) (layers *.Cu *.Mask))
-    (pad "" np_thru_hole circle (at 12.155 7.32 180) (size 5.57 5.57) (drill 4.57) (layers *.Cu *.Mask))
-    (pad 1 thru_hole circle (at -3.95 15.8 180) (size 3 3) (drill 1.8) (layers *.Cu *.Mask)
-      (net 47 "Net-(J1-Pad1)"))
-    (pad 2 thru_hole circle (at 3.95 15.8 180) (size 3 3) (drill 1.8) (layers *.Cu *.Mask)
-      (net 2 GND))
-  )
   (gr_text LFXTL (at 149.86 57.15 90) (layer F.Mask)
     (effects (font (size 1.4478 1.016) (thickness 0.254)))
@@
   (segment (start 136.5504 54.61) (end 136.6774 54.483) (width 0.3) (layer F.Cu) (net 2))
   (segment (start 135.89 54.61) (end 136.5504 54.61) (width 0.3) (layer F.Cu) (net 2))
-  (segment (start 139.9286 54.483) (end 139.9286 55.6006) (width 0.3) (layer F.Cu) (net 2))
-  (segment (start 140.589 54.483) (end 140.589 55.499) (width 0.3) (layer F.Cu) (net 2))
   (segment (start 136.6774 54.483) (end 136.6774 53.1114) (width 0.3) (layer F.Cu) (net 2))
   (segment (start 135.255 33.655) (end 133.985 33.655) (width 0.3) (layer F.Cu) (net 2))
@@
   (segment (start 132.08 59.055) (end 132.08 61.595) (width 0.3) (layer B.Cu) (net 2))
   (segment (start 135.89 54.61) (end 132.08 58.42) (width 0.3) (layer B.Cu) (net 2))
-  (segment (start 67.17 151.84) (end 70.778 155.448) (width 2.032) (layer F.Cu) (net 2))
-  (segment (start 70.778 155.448) (end 82.55 155.448) (width 2.032) (layer F.Cu) (net 2))
-  (segment (start 82.55 155.448) (end 102.616 155.448) (width 2.032) (layer F.Cu) (net 2))
+  (segment (start 75.07 151.84) (end 104.065 151.84) (width 2.032) (layer F.Cu) (net 2))
   (segment (start 105.918 82.55) (end 103.285 82.55) (width 0.508) (layer F.Cu) (net 3))
   (segment (start 103.285 82.55) (end 91.855 93.98) (width 0.508) (layer F.Cu) (net 3))
@@
   (segment (start 99.06 137.16) (end 54.61 137.16) (width 1.016) (layer F.Cu) (net 47))
   (segment (start 54.435 134.21) (end 54.435 140.11) (width 2.032) (layer F.Cu) (net 47))
-  (segment (start 54.435 140.11) (end 69.498 140.11) (width 2.032) (layer F.Cu) (net 47))
-  (segment (start 75.07 145.682) (end 75.07 151.84) (width 2.032) (layer F.Cu) (net 47))
-  (segment (start 69.498 140.11) (end 75.07 145.682) (width 2.032) (layer F.Cu) (net 47))
+  (segment (start 54.435 140.11) (end 60.735 140.11) (width 2.032) (layer F.Cu) (net 47))
+  (segment (start 67.17 146.545) (end 67.17 151.84) (width 2.032) (layer F.Cu) (net 47))
+  (segment (start 60.735 140.11) (end 67.17 146.545) (width 2.032) (layer F.Cu) (net 47))
   (via (at 136.8044 56.007) (size 0.8) (drill 0.4) (layers F.Cu B.Cu) (net 48))
   (segment (start 137.3124 55.499) (end 136.8044 56.007) (width 0.3) (layer F.Cu) (net 48))
