File: projects/Battery-Experiments/Avionics Battery Prototype/XTAL plug/XTAL plug.sch (KiCad schematic (older format))
At the start: 2 parts, among them J1 Conn_01x02, X1 Crystal

Commit message: AVB Rev C and XTAL Plug Final
Parts:
- J1: footprint Connector_PinSocket_2.54mm:PinSocket_1x02_P2.54mm_Vertical -> k7arx:PreciDip 8MM-11 2-pin SMD
Changed lines of the file:
@@
 F 0 "J1" V 5514 3262 50  0000 R CNN
 F 1 "Conn_01x02" V 5423 3262 50  0000 R CNN
-F 2 "Connector_PinSocket_2.54mm:PinSocket_1x02_P2.54mm_Vertical" H 5550 3450 50  0001 C CNN
+F 2 "k7arx:PreciDip 8MM-11 2-pin SMD" H 5550 3450 50  0001 C CNN
 F 3 "~" H 5550 3450 50  0001 C CNN
 	1    5550 3450
